File: Schematic and PCB/RF_Switch_module.sch (KiCad schematic (older format))
At the start: 21 parts, among them J1 Conn_01x01, J2 Conn_01x04, Q1 IRF740, SW1 SW_Push, U1 SYN480R, U2 RFE272A, U3 L7805, Y1 6.7458MHz

Commit message: Routing
Parts:
- C1, C2, C3, C4, C5, C6, C7: footprint Capacitor_SMD:C_01005_0402Metric -> Capacitor_SMD:C_0402_1005Metric
- C8: footprint Capacitor_SMD:C_1206_3216Metric -> Capacitor_SMD:C_0402_1005Metric
- J2: footprint Connector_PinHeader_2.54mm:PinHeader_1x04_P2.54mm_Horizontal -> Connector_PinHeader_2.54mm_OSHW:PinHeader_1x04_P2.54mm_Horizontal
- Q1: footprint Package_TO_SOT_THT:TO-220-3_Vertical -> Package_TO_SOT_SMD:TO-252-3_TabPin2
- R1, R2: footprint Resistor_SMD:R_01005_0402Metric -> Resistor_SMD:R_0402_1005Metric
- SW1: footprint Button_Switch_SMD:SW_DIP_SPSTx01_Slide_6.7x4.1mm_W6.73mm_P2.54mm_LowProfile_JPin -> Button_Switch_SMD:SW_Push_SPST_NO_Alps_SKRK
Changed lines of the file:
@@
 F 0 "R1" H 7320 4146 50  0000 L CNN
 F 1 "2.2KOhm" H 7320 4055 50  0000 L CNN
-F 2 "Resistor_SMD:R_01005_0402Metric" V 7180 4100 50  0001 C CNN
+F 2 "Resistor_SMD:R_0402_1005Metric" V 7180 4100 50  0001 C CNN
 F 3 "~" H 7250 4100 50  0001 C CNN
 	1    7250 4100
@@
 F 0 "SW1" V 6246 4052 50  0000 R CNN
 F 1 "SW_Push" V 6155 4052 50  0000 R CNN
-F 2 "Button_Switch_SMD:SW_DIP_SPSTx01_Slide_6.7x4.1mm_W6.73mm_P2.54mm_LowProfile_JPin" H 6200 4300 50  0001 C CNN
+F 2 "Button_Switch_SMD:SW_Push_SPST_NO_Alps_SKRK" H 6200 4300 50  0001 C CNN
 F 3 "~" H 6200 4300 50  0001 C CNN
 	1    6200 4100
@@
 F 0 "C6" H 6765 2746 50  0000 L CNN
 F 1 "4.7uF" H 6765 2655 50  0000 L CNN
-F 2 "Capacitor_SMD:C_01005_0402Metric" H 6688 2550 50  0001 C CNN
+F 2 "Capacitor_SMD:C_0402_1005Metric" H 6688 2550 50  0001 C CNN
 F 3 "~" H 6650 2700 50  0001 C CNN
 	1    6650 2700
@@
 F 0 "C5" H 6265 2746 50  0000 L CNN
 F 1 "0.01uF" H 6265 2655 50  0000 L CNN
-F 2 "Capacitor_SMD:C_01005_0402Metric" H 6188 2550 50  0001 C CNN
+F 2 "Capacitor_SMD:C_0402_1005Metric" H 6188 2550 50  0001 C CNN
 F 3 "~" H 6150 2700 50  0001 C CNN
 	1    6150 2700
@@
 F 0 "R2" V 6843 3750 50  0000 C CNN
 F 1 "1.2KOhm" V 6934 3750 50  0000 C CNN
-F 2 "Resistor_SMD:R_01005_0402Metric" V 6980 3750 50  0001 C CNN
+F 2 "Resistor_SMD:R_0402_1005Metric" V 6980 3750 50  0001 C CNN
 F 3 "~" H 7050 3750 50  0001 C CNN
 	1    7050 3750
@@
 F 0 "Q1" H 8206 3796 50  0000 L CNN
 F 1 "IRF740" H 8206 3705 50  0000 L CNN
-F 2 "Package_TO_SOT_THT:TO-220-3_Vertical" H 8250 3675 50  0001 L CIN
+F 2 "Package_TO_SOT_SMD:TO-252-3_TabPin2" H 8250 3675 50  0001 L CIN
 F 3 "http://www.vishay.com/docs/91054/91054.pdf" H 8000 3750 50  0001 L CNN
 	1    8000 3750
@@
 F 0 "C1" H 2815 3446 50  0000 L CNN
 F 1 "8.2pF" H 2815 3355 50  0000 L CNN
-F 2 "Capacitor_SMD:C_01005_0402Metric" H 2738 3250 50  0001 C CNN
+F 2 "Capacitor_SMD:C_0402_1005Metric" H 2738 3250 50  0001 C CNN
 F 3 "~" H 2700 3400 50  0001 C CNN
 	1    2700 3400
@@
 F 0 "C3" H 3565 3896 50  0000 L CNN
 F 1 "2.2uF" H 3565 3805 50  0000 L CNN
-F 2 "Capacitor_SMD:C_01005_0402Metric" H 3488 3700 50  0001 C CNN
+F 2 "Capacitor_SMD:C_0402_1005Metric" H 3488 3700 50  0001 C CNN
 F 3 "~" H 3450 3850 50  0001 C CNN
 	1    3450 3850
@@
 F 0 "C2" H 3215 3646 50  0000 L CNN
 F 1 "4.7uF" H 3215 3555 50  0000 L CNN
-F 2 "Capacitor_SMD:C_01005_0402Metric" H 3138 3450 50  0001 C CNN
+F 2 "Capacitor_SMD:C_0402_1005Metric" H 3138 3450 50  0001 C CNN
 F 3 "~" H 3100 3600 50  0001 C CNN
 	1    3100 3600
@@
 F 0 "C4" V 4548 3050 50  0000 C CNN
 F 1 "4.7uF" V 4639 3050 50  0000 C CNN
-F 2 "Capacitor_SMD:C_01005_0402Metric" H 4838 2900 50  0001 C CNN
+F 2 "Capacitor_SMD:C_0402_1005Metric" H 4838 2900 50  0001 C CNN
 F 3 "~" H 4800 3050 50  0001 C CNN
 	1    4800 3050
@@
 F 0 "C7" H 5315 5196 50  0000 L CNN
 F 1 "0.33uF" H 5315 5105 50  0000 L CNN
-F 2 "Capacitor_SMD:C_01005_0402Metric" H 5238 5000 50  0001 C CNN
+F 2 "Capacitor_SMD:C_0402_1005Metric" H 5238 5000 50  0001 C CNN
 F 3 "~" H 5200 5150 50  0001 C CNN
 	1    5200 5150
@@
 F 0 "C8" H 6215 5196 50  0000 L CNN
 F 1 "0.1uF" H 6215 5105 50  0000 L CNN
-F 2 "Capacitor_SMD:C_1206_3216Metric" H 6138 5000 50  0001 C CNN
+F 2 "Capacitor_SMD:C_0402_1005Metric" H 6138 5000 50  0001 C CNN
 F 3 "~" H 6100 5150 50  0001 C CNN
 	1    6100 5150
@@
 F 0 "J2" H 9380 3042 50  0000 L CNN
 F 1 "Conn_01x04" H 9380 2951 50  0000 L CNN
-F 2 "Connector_PinHeader_2.54mm:PinHeader_1x04_P2.54mm_Horizontal" H 9300 3050 50  0001 C CNN
+F 2 "Connector_PinHeader_2.54mm_OSHW:PinHeader_1x04_P2.54mm_Horizontal" H 9300 3050 50  0001 C CNN
 F 3 "~" H 9300 3050 50  0001 C CNN
 	1    9300 3050
