File: Schematic and PCB/RF_Switch_module.kicad_pcb (KiCad board)
At the start: 2 copper layers, 21 parts, among them J1 Conn_01x01, J2 Conn_01x04, Q1 IRF740, SW1 SW_Push, U1 SYN480R, U2 RFE272A, U3 L7805, Y1 6.7458MHz

Commit message: Routing
Routing:
- added copper zone on B.Cu, net GND
- added copper zone on F.Cu, net GND
Other:
- board outline added: 28.7 x 11.7 mm
Changed lines of the file:
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@@
   (general
     (thickness 1.6)
-    (drawings 0)
+    (drawings 7)
     (tracks 132)
     (zones 0)
@@
   )
   (page A4)
+  (title_block
+    (title RF_Switch_module)
+    (date 2019-05-13)
+    (rev 0.1)
+    (company OSHW)
+  )
   (layers
     (0 F.Cu signal)
@@
     (add_net VDD)
   )
+  (module Crystal:Crystal_HC49-U_Vertical (layer F.Cu)
+    (at 168.91 102.235)
+    (descr "Crystal THT HC-49/U http://5hertz.com/pdfs/04404_D.pdf")
+    (tags "THT crystalHC-49/U")
+    (fp_text reference Y1 (at 2.44 -3.525) (layer F.SilkS)
+      (effects (font (size 1 1) (thickness 0.15)))
+    )
+    (fp_text value 6.7458MHz (at 2.44 3.525) (layer F.Fab)
+      (effects (font (size 1 1) (thickness 0.15)))
+    )
+    (fp_text user %R (at 2.44 0) (layer F.Fab)
+      (effects (font (size 1 1) (thickness 0.15)))
+    )
+    (fp_line (start -0.685 -2.325) (end 5.565 -2.325) (layer F.Fab) (width 0.1))
+    (fp_line (start -0.685 2.325) (end 5.565 2.325) (layer F.Fab) (width 0.1))
+    (fp_line (start -0.56 -2) (end 5.44 -2) (layer F.Fab) (width 0.1))
+    (fp_line (start -0.56 2) (end 5.44 2) (layer F.Fab) (width 0.1))
+    (fp_line (start -0.685 -2.525) (end 5.565 -2.525) (layer F.SilkS) (width 0.12))
+    (fp_line (start -0.685 2.525) (end 5.565 2.525) (layer F.SilkS) (width 0.12))
+    (fp_line (start -3.5 -2.8) (end -3.5 2.8) (layer F.CrtYd) (width 0.05))
+    (fp_line (start -3.5 2.8) (end 8.4 2.8) (layer F.CrtYd) (width 0.05))
+    (fp_line (start 8.4 2.8) (end 8.4 -2.8) (layer F.CrtYd) (width 0.05))
+    (fp_line (start 8.4 -2.8) (end -3.5 -2.8) (layer F.CrtYd) (width 0.05))
+    (fp_arc (start -0.685 0) (end -0.685 -2.325) (angle -180) (layer F.Fab) (width 0.1))
+    (fp_arc (start 5.565 0) (end 5.565 -2.325) (angle 180) (layer F.Fab) (width 0.1))
+    (fp_arc (start -0.56 0) (end -0.56 -2) (angle -180) (layer F.Fab) (width 0.1))
+    (fp_arc (start 5.44 0) (end 5.44 -2) (angle 180) (layer F.Fab) (width 0.1))
+    (fp_arc (start -0.685 0) (end -0.685 -2.525) (angle -180) (layer F.SilkS) (width 0.12))
+    (fp_arc (start 5.565 0) (end 5.565 -2.525) (angle 180) (layer F.SilkS) (width 0.12))
+    (pad 1 thru_hole circle (at 0 0) (size 1.5 1.5) (drill 0.8) (layers *.Cu *.Mask)
+      (net 2 GND))
+    (pad 2 thru_hole circle (at 4.88 0) (size 1.5 1.5) (drill 0.8) (layers *.Cu *.Mask)
+      (net 12 "Net-(U1-Pad8)"))
+    (model ${KISYS3DMOD}/Crystal.3dshapes/Crystal_HC49-U_Vertical.wrl
+      (at (xyz 0 0 0))
+      (scale (xyz 1 1 1))
+      (rotate (xyz 0 0 0))
+    )
+  )
   (module LED_SMD:LED_0402_1005Metric (layer B.Cu)
     (at 173.505 104.14 180)
@@
       (net 2 GND))
     (model ${KISYS3DMOD}/Package_TO_SOT_SMD.3dshapes/SOT-89-3.wrl
-      (at (xyz 0 0 0))
-      (scale (xyz 1 1 1))
-      (rotate (xyz 0 0 0))
-    )
-  )
-  (module Crystal:Crystal_HC49-U_Vertical (layer F.Cu)
-    (at 168.91 102.235)
-    (descr "Crystal THT HC-49/U http://5hertz.com/pdfs/04404_D.pdf")
-    (tags "THT crystalHC-49/U")
-    (fp_text reference Y1 (at 2.44 -3.525) (layer F.SilkS)
-      (effects (font (size 1 1) (thickness 0.15)))
-    )
-    (fp_text value 6.7458MHz (at 2.44 3.525) (layer F.Fab)
-      (effects (font (size 1 1) (thickness 0.15)))
-    )
-    (fp_text user %R (at 2.44 0) (layer F.Fab)
-      (effects (font (size 1 1) (thickness 0.15)))
-    )
-    (fp_line (start -0.685 -2.325) (end 5.565 -2.325) (layer F.Fab) (width 0.1))
-    (fp_line (start -0.685 2.325) (end 5.565 2.325) (layer F.Fab) (width 0.1))
-    (fp_line (start -0.56 -2) (end 5.44 -2) (layer F.Fab) (width 0.1))
-    (fp_line (start -0.56 2) (end 5.44 2) (layer F.Fab) (width 0.1))
-    (fp_line (start -0.685 -2.525) (end 5.565 -2.525) (layer F.SilkS) (width 0.12))
-    (fp_line (start -0.685 2.525) (end 5.565 2.525) (layer F.SilkS) (width 0.12))
-    (fp_line (start -3.5 -2.8) (end -3.5 2.8) (layer F.CrtYd) (width 0.05))
-    (fp_line (start -3.5 2.8) (end 8.4 2.8) (layer F.CrtYd) (width 0.05))
-    (fp_line (start 8.4 2.8) (end 8.4 -2.8) (layer F.CrtYd) (width 0.05))
-    (fp_line (start 8.4 -2.8) (end -3.5 -2.8) (layer F.CrtYd) (width 0.05))
-    (fp_arc (start -0.685 0) (end -0.685 -2.325) (angle -180) (layer F.Fab) (width 0.1))
-    (fp_arc (start 5.565 0) (end 5.565 -2.325) (angle 180) (layer F.Fab) (width 0.1))
-    (fp_arc (start -0.56 0) (end -0.56 -2) (angle -180) (layer F.Fab) (width 0.1))
-    (fp_arc (start 5.44 0) (end 5.44 -2) (angle 180) (layer F.Fab) (width 0.1))
-    (fp_arc (start -0.685 0) (end -0.685 -2.525) (angle -180) (layer F.SilkS) (width 0.12))
-    (fp_arc (start 5.565 0) (end 5.565 -2.525) (angle 180) (layer F.SilkS) (width 0.12))
-    (pad 1 thru_hole circle (at 0 0) (size 1.5 1.5) (drill 0.8) (layers *.Cu *.Mask)
-      (net 2 GND))
-    (pad 2 thru_hole circle (at 4.88 0) (size 1.5 1.5) (drill 0.8) (layers *.Cu *.Mask)
-      (net 12 "Net-(U1-Pad8)"))
-    (model ${KISYS3DMOD}/Crystal.3dshapes/Crystal_HC49-U_Vertical.wrl
       (at (xyz 0 0 0))
       (scale (xyz 1 1 1))
@@
     )
   )
+  (gr_line (start 191.008 99.568) (end 162.306 99.568) (layer Edge.Cuts) (width 0.05))
+  (gr_line (start 191.008 111.252) (end 191.008 99.568) (layer Edge.Cuts) (width 0.05))
+  (gr_line (start 179.832 111.252) (end 191.008 111.252) (layer Edge.Cuts) (width 0.05))
+  (gr_line (start 162.306 111.252) (end 179.832 111.252) (layer Edge.Cuts) (width 0.05))
+  (gr_line (start 162.306 110.998) (end 162.306 111.252) (layer Edge.Cuts) (width 0.05))
+  (gr_line (start 162.306 110.744) (end 162.306 110.998) (layer Edge.Cuts) (width 0.05))
+  (gr_line (start 162.306 99.568) (end 162.306 110.744) (layer Edge.Cuts) (width 0.05))
   (segment (start 163.345 104.14) (end 163.345 105.41) (width 0.25) (layer F.Cu) (net 1))
   (segment (start 163.345 105.41) (end 163.345 106.195) (width 0.25) (layer F.Cu) (net 1))
@@
   (segment (start 172.72 109.855) (end 174.025 109.855) (width 0.25) (layer F.Cu) (net 13))
   (segment (start 168.875 108.585) (end 167.9 108.585) (width 0.25) (layer B.Cu) (net 15))
+  (zone (net 2) (net_name GND) (layer B.Cu) (hatch edge 0.508)
+    (connect_pads (clearance 0.508))
+    (min_thickness 0.254)
+    (fill yes (arc_segments 32) (thermal_gap 0.508) (thermal_bridge_width 0.508))
+    (polygon
+      (pts
+        (xy 162.306 99.568) (xy 162.306 111.252) (xy 191.008 111.252) (xy 191.008 99.568)
+      )
+    )
+  )
+  (zone (net 2) (net_name GND) (layer F.Cu) (hatch edge 0.508)
+    (connect_pads (clearance 0.508))
+    (min_thickness 0.254)
+    (fill yes (arc_segments 32) (thermal_gap 0.508) (thermal_bridge_width 0.508))
+    (polygon
+      (pts
+        (xy 162.306 99.568) (xy 162.306 111.252) (xy 191.008 111.252) (xy 191.008 99.568)
+      )
+    )
+  )
 )
